File: C64 Mega Switcher.kicad_pcb (KiCad board)
At the start: 2 copper layers, 44.2 x 81.5 mm, 25 parts, among them J1 Port 1, J2 Port 2, J3 Mega Drive, J4 C_SEL, J5 B_SEL, SW1 P1_SEL, SW2 P2_SEL, U1 74HCT4053, U2 74HCT4053, U3 NE555

Commit message: Revision B
Parts:
- added D10: 1N4148, Diodes_THT:D_DO-35_SOD27_P2.54mm_Vertical_AnodeUp, F.Cu at (113.7, 84.5)
- added D11: 1N4148, Diodes_THT:D_DO-35_SOD27_P2.54mm_Vertical_AnodeUp, F.Cu at (113.7, 56.5)
- added D12: 1N4148, Diodes_THT:D_DO-35_SOD27_P2.54mm_Vertical_AnodeUp, F.Cu at (113.7, 87.6)
- added D8: 1N4148, Diodes_THT:D_DO-35_SOD27_P2.54mm_Vertical_AnodeUp, F.Cu at (113.7, 81.3)
- added D9: 1N4148, Diodes_THT:D_DO-35_SOD27_P2.54mm_Vertical_AnodeUp, F.Cu at (113.7, 53.3)
- added Q1: BC547, TO_SOT_Packages_THT:TO-92_Inline_Wide, F.Cu at (112.4, 64.8)
- added R5: 2k2, Resistors_THT:R_Axial_DIN0207_L6.3mm_D2.5mm_P10.16mm_Horizontal, F.Cu at (118.7, 67.3)
- added R6: 100k, Resistors_THT:R_Axial_DIN0207_L6.3mm_D2.5mm_P10.16mm_Horizontal, F.Cu at (118.7, 71.1)
- added R7: 2k2, Resistors_THT:R_Axial_DIN0207_L6.3mm_D2.5mm_P10.16mm_Horizontal, F.Cu at (118.7, 74.9)
- J4, J5: footprint Pin_Headers:Pin_Header_Straight_2x02_Pitch2.54mm -> Pin_Headers:Pin_Header_Straight_2x03_Pitch2.54mm
- moved D3 58.7 mm to (113.7, 43.8), turned to 180 degrees
- moved D5 55.3 mm to (113.7, 47.0), turned to 180 degrees
- moved D7 53.4 mm to (113.7, 50.2), turned to 180 degrees
- moved U2 43.3 mm to (134.6, 41.3)
- moved C2 42.7 mm to (141.0, 37.5), turned to 180 degrees
- moved R4 31.2 mm to (118.7, 82.5), turned to 0 degrees
- moved D6 28.9 mm to (113.7, 78.1), turned to 180 degrees
- moved D4 27.4 mm to (113.7, 74.9), turned to 180 degrees
- moved R3 25.8 mm to (118.7, 78.7), turned to 0 degrees
- moved R2 24.6 mm to (133.3, 82.5), turned to 0 degrees
- moved U3 22.5 mm to (134.6, 67.3)
- moved R1 21.7 mm to (133.3, 78.7), turned to 0 degrees
- moved J5 21.0 mm to (114.3, 95.2)
- moved C3 17.4 mm to (141.0, 63.5), turned to 180 degrees
- moved SW2 15.4 mm to (141.0, 115.6), turned to 90 degrees
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Connections:
- net /MD_U renamed /MD_UP
- D3 pad 1: /MD_R -> Net-(D3-Pad1)
- D3 pad 2: RIGHT -> Net-(D3-Pad2)
- D4 pad 1: /MD_L -> Net-(D4-Pad1)
- D4 pad 2: LEFT -> Net-(D4-Pad2)
- D5 pad 1: /MD_D -> Net-(D5-Pad1)
- D5 pad 2: DOWN -> Net-(D5-Pad2)
- D6 pad 2: FIRE -> Net-(D6-Pad2)
- D7 pad 2: UP -> Net-(D7-Pad2)
- J1 pad 1: Net-(J1-Pad1) -> Net-(D12-Pad2)
- J1 pad 2: Net-(J1-Pad2) -> Net-(D8-Pad2)
- J1 pad 3: Net-(J1-Pad3) -> Net-(D6-Pad2)
- J1 pad 4: Net-(J1-Pad4) -> Net-(D4-Pad2)
- J1 pad 6: Net-(J1-Pad6) -> Net-(D10-Pad2)
- J1 pad 9: (no net) -> Net-(J1-Pad9)
- J2 pad 1: Net-(J2-Pad1) -> Net-(D11-Pad2)
- J2 pad 2: Net-(J2-Pad2) -> Net-(D7-Pad2)
- J2 pad 3: Net-(J2-Pad3) -> Net-(D5-Pad2)
- J2 pad 4: Net-(J2-Pad4) -> Net-(D3-Pad2)
- J2 pad 6: Net-(J2-Pad6) -> Net-(D9-Pad2)
- J2 pad 9: (no net) -> Net-(J2-Pad9)
- J3 pad 2: /MD_D -> DOWN
- J3 pad 3: /MD_L -> LEFT
- J3 pad 4: /MD_R -> RIGHT
- J3 pad 6: Net-(J3-Pad6) -> /MD_BTN_B
- J3 pad 9: Net-(J3-Pad9) -> /MD_BTN_C
- J4 pad 1: Net-(J3-Pad9) -> /MD_BTN_C
- J4 pad 2: Net-(D7-Pad1) -> UP
- J4 pad 3: Net-(J3-Pad9) -> /MD_BTN_C
- J4 pad 4: Net-(D6-Pad1) -> FIRE
- J5 pad 1: Net-(J3-Pad6) -> /MD_BTN_B
- J5 pad 2: Net-(D7-Pad1) -> UP
- J5 pad 3: Net-(J3-Pad6) -> /MD_BTN_B
- J5 pad 4: Net-(D6-Pad1) -> FIRE
- JP1 pad 1: Net-(D7-Pad1) -> UP
- R1 pad 1: VCC -> Net-(R1-Pad1)
- R1 pad 2: Net-(R1-Pad2) -> VCC
- R2 pad 1: VCC -> Net-(R2-Pad1)
- R2 pad 2: Net-(R2-Pad2) -> VCC
- R3 pad 1: VCC -> Net-(D1-Pad2)
- R3 pad 2: Net-(D1-Pad2) -> VCC
- R4 pad 1: Net-(D2-Pad1) -> GND
- R4 pad 2: GND -> Net-(D2-Pad1)
- SW1 pad 2: Net-(R2-Pad2) -> Net-(R2-Pad1)
- SW2 pad 2: Net-(R1-Pad2) -> Net-(R1-Pad1)
- U1 pad 1: Net-(J1-Pad3) -> Net-(D6-Pad1)
- U1 pad 12: Net-(J2-Pad4) -> Net-(D3-Pad1)
- U1 pad 13: Net-(J1-Pad4) -> Net-(D4-Pad1)
- U1 pad 2: Net-(J2-Pad3) -> Net-(D5-Pad1)
- U1 pad 3: Net-(J1-Pad2) -> Net-(D8-Pad1)
- U1 pad 5: Net-(J2-Pad2) -> Net-(D7-Pad1)
- U2 pad 1: Net-(J1-Pad1) -> Net-(D12-Pad1)
- U2 pad 12: Net-(J2-Pad6) -> Net-(D9-Pad1)
- U2 pad 13: Net-(J1-Pad6) -> Net-(D10-Pad1)
- U2 pad 2: Net-(J2-Pad1) -> Net-(D11-Pad1)
- U2 pad 3: (no net) -> Net-(J1-Pad9)
- U2 pad 4: GND -> ALT_FIRE
- U2 pad 5: (no net) -> Net-(J2-Pad9)
- U3 pad 2: Net-(R2-Pad2) -> Net-(R2-Pad1)
- U3 pad 4: Net-(R1-Pad2) -> Net-(R1-Pad1)
Routing:
- net Net-(R2-Pad2): track 87.4 -> 0.00 mm, vias 1 -> 0
- net Net-(R1-Pad2): track 77.6 -> 0.00 mm
- net Net-(D12-Pad1): track 0.00 -> 69.9 mm, vias 0 -> 4
- net Net-(D8-Pad1): track 0.00 -> 69.6 mm, vias 0 -> 4
- net Net-(D10-Pad1): track 0.00 -> 63.0 mm, vias 0 -> 4
- net UP: track 29.0 -> 89.3 mm
- net Net-(J2-Pad6): track 60.1 -> 0.00 mm
- net Net-(J1-Pad9): track 0.00 -> 59.2 mm, vias 0 -> 6
- net FIRE: track 29.0 -> 85.3 mm
- net Net-(R1-Pad1): track 0.00 -> 56.1 mm, vias 0 -> 2
- net Net-(R2-Pad1): track 0.00 -> 51.9 mm, vias 0 -> 2
- net Net-(J1-Pad3): track 49.3 -> 0.00 mm, vias 4 -> 0
- net Net-(J1-Pad2): track 48.9 -> 0.00 mm
- net Net-(J3-Pad6): track 48.0 -> 0.00 mm, vias 4 -> 0
- net ALT_FIRE: track 0.00 -> 44.4 mm, vias 0 -> 5
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Other:
- board size 44.2 x 81.5 mm -> 49.3 x 81.5 mm
- board text added: "ALT"
- board text added: "B"
- board text added: "C"
- board text added: "D-UP"
- board text added: "Do NOT change when powered, do not jumper more than once per line!"
- board text added: "Licensed under CERN OHL v.1.2"
- board text added: "Revision B"
- board text added: "github.com/tebl"
- board text removed: "B SELECT"
- board text removed: "C SELECT"
- board text removed: "D-PAD UP"
- board text removed: "Do NOT change when powered, do not jumper any function MORE than ONCE!"
- board text removed: "Enable"
- board text removed: "Licensed under CERN OHL v.1.2 github.com/tebl"
- board text removed: "WARNING! Read documentation!"
